File: sdmmc.kicad_sch (KiCad schematic)
At the start: 0 parts

Commit message: Added SDMMC
Parts:
- added C3: 4.7nF, Capacitor_SMD:C_0805_2012Metric_Pad1.18x1.45mm_HandSolder, symbol Device:C_Small
- added J4: MSD-4-A, MSD_4_A:CUI_MSD-4-A, symbol MSD-4-A:MSD-4-A
- added R12: R, Resistor_SMD:R_0805_2012Metric_Pad1.20x1.40mm_HandSolder, symbol Device:R
- added R13: 1MΩ, Resistor_SMD:R_0805_2012Metric_Pad1.20x1.40mm_HandSolder, symbol Device:R
Connections:
- new net: C3.2, J4.G1 (COVER_GND), J4.G2 (COVER_GND__1), J4.G3 (COVER_GND__2), J4.G4 (COVER_GND__3), R13.1
- new net +3V3: J4.4 (VDD), R12.1
- new net GND: C3.1, J4.6 (VSS), R13.2
- new net SDMMC_CLK: J4.5 (CLK)
- new net SDMMC_CMD: J4.3 (CMD)
- new net SDMMC_DAT0: J4.7 (DAT0)
- new net SDMMC_DAT1: J4.8 (DAT1)
- new net SDMMC_DAT2: J4.1 (DAT2)
- new net SDMMC_DAT3: J4.2 (CD/DAT3)
- new net SDMMC_nDET: J4.CD, R12.2
