File: ethernet.kicad_sch (KiCad schematic)
At the start: 47 parts, among them J1 SI-52008-F, U2 LAN8742A, Y1 ECS-3225MVLC-500-CN-TR

Commit message: Started with pin mapping
Parts:
- L1: footprint (none) -> Inductor_SMD:L_0805_2012Metric_Pad1.05x1.20mm_HandSolder
Changed lines of the file:
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@@
 			)
 		)
-		(property "Footprint" ""
+		(property "Footprint" "Inductor_SMD:L_0805_2012Metric_Pad1.05x1.20mm_HandSolder"
 			(at 114.3 35.56 0)
 			(effects

Commit message: layout v1
no silkscreen done yet
Parts:
- removed R24: 33R, Resistor_SMD:R_0805_2012Metric_Pad1.20x1.40mm_HandSolder, symbol Device:R
Connections:
- net ETH_RXER: now also U2.10 (RXER/PHYAD0)
Changed lines of the file:
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@@
 	(wire
 		(pts
-			(xy 73.66 101.6) (xy 76.2 101.6)
-		)
-		(stroke
-			(width 0)
-			(type default)
-		)
-	)
-	(wire
-		(pts
 			(xy 114.3 82.55) (xy 119.38 82.55)
 		)
@@
 	(wire
 		(pts
-			(xy 63.5 101.6) (xy 66.04 101.6)
+			(xy 63.5 101.6) (xy 76.2 101.6)
 		)
 		(stroke
@@
 					(unit 1)
 				)
-			)
-		)
-	)
-	(symbol
-		(lib_id "Device:R")
-		(at 69.85 101.6 270)
-		(mirror x)
-		(unit 1)
-		(exclude_from_sim no)
-		(in_bom yes)
-		(on_board yes)
-		(dnp no)
-		(property "Reference" "R24"
-			(at 69.85 105.918 90)
-			(effects
-				(font
-					(size 1.27 1.27)
-				)
-				(hide yes)
-			)
-		)
-		(property "Value" "33R"
-			(at 69.85 103.886 90)
-			(effects
-				(font
-					(size 1.27 1.27)
-				)
-			)
-		)
-		(property "Footprint" "Resistor_SMD:R_0805_2012Metric_Pad1.20x1.40mm_HandSolder"
-			(at 69.85 103.378 90)
-			(effects
-				(font
-					(size 1.27 1.27)
-				)
-				(hide yes)
-			)
-		)
-		(property "Datasheet" "~"
-			(at 69.85 101.6 0)
-			(effects
-				(font
-					(size 1.27 1.27)
-				)
-				(hide yes)
-			)
-		)
-		(property "Description" "Resistor"
-			(at 69.85 101.6 0)
-			(effects
-				(font
-					(size 1.27 1.27)
-				)
-				(hide yes)
-			)
-		)
-		(pin "1"
-		)
-		(pin "2"
-		)
-		(instances
-			(project "miniServer"
-				(path "/2f7e2d6e-7ac1-4ae5-be0e-a6d141d8b943/5bc2eac8-7f57-4126-99be-333aeb01e149"
-					(reference "R24")
-					(unit 1)
-				)

Commit message: Changed ETH connector, cleared old layout
Parts:
- removed J1: SI-52008-F, SI_52008_F:BEL_SI-52008-F, symbol SI_52008_F:SI-52008-F
- added J5: 0826-1X1T-GJ-F, 0826-1X1T-GJ-F:BEL_0826-1X1T-GJ-F, symbol 0826-1X1T-GJ-F:0826-1X1T-GJ-F
Connections:
- net +3V3: now also J5.17
- net GND: now also J5.20
- net VDDA: now also J5.12 (TRCT1), J5.6 (TRCT2)
- net at D10.2 (A), D9.1 (K): now also J5.16 (VC78)
- net at C10.2, R21.1, U2.21 (TXP): now also J5.11 (TRD1+)
- net at C11.2, R20.1, U2.20 (TXN): now also J5.10 (TRD1-)
- net at C13.2, R18.1, U2.22 (RXN): now also J5.5 (TRD2-)
- net at C12.2, R19.1, U2.23 (RXP): now also J5.4 (TRD2+)
- net at D6.1 (K), D8.2 (A): now also J5.15 (VC45)
- net at D4.1 (K), D7.2 (A): now also J5.13 (VC12)
- net at C4.2, R14.1: now also J5.S1 (SHIELD), J5.S2 (SHIELD__1)
- net at D3.2 (A), D5.1 (K): now also J5.14 (VC36)
- net at R5.2: now also J5.19
- net at R4.2: now also J5.18
Other:
- moved on the sheet: R25, R4, R5, R8

Commit message: Changed PowerSupply idea: use jumper to select PoE or VBUS
Parts:
- removed C14: 22uF, Capacitor_SMD:C_0805_2012Metric_Pad1.18x1.45mm_HandSolder, symbol Device:C_Small
- removed C15: 330uF, Capacitor_SMD:C_0805_2012Metric_Pad1.18x1.45mm_HandSolder, symbol Device:C_Small
- removed D10, D3, D4, D5, D6, D7, D8, D9: D_Schottky, Diode_SMD:Nexperia_CFP3_SOD-123W, symbol Device:D_45deg
- removed D11: D_Schottky, Diode_SMD:Nexperia_CFP3_SOD-123W, symbol Device:D_Schottky
- removed MD1: MURATA_MYBSP00502ABF, MYBSP00502ABF:MURATA_MYBSP00502ABF_0, symbol MURATA_MYBSP00502ABF:MURATA_MYBSP00502ABF
- added D1: WE-TVS_SOT23-6L_82402305, WE-TVS_SOT23-6L_82402305:WE-TVS_SOT23-6L, symbol WE-TVS_SOT23-6L_82402305:WE-TVS_SOT23-6L_82402305
Connections:
- net GND: now also D1.2
- net VDDA: now also D1.5
- net PoE/V2-: now reaches J5.16 (VC78)
- net at C10.2, J5.11 (TRD1+), R21.1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: now also D1.3
- net at C11.2, J5.10 (TRD1-), R20.1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: now also D1.1
- net at C13.2, J5.5 (TRD2-), R18.1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: now also D1.4
- net at C12.2, J5.4 (TRD2+), R19.1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: now also D1.6
- net PoE/V2+: now reaches J5.15 (VC45)
- net PoE/V1+: now reaches J5.13 (VC12)
- net PoE/V1-: now reaches J5.14 (VC36)
Other:
- added sheet PoE (PoE.kicad_sch)
- moved on the sheet: C10, C11, C12, C13, C2, C4, C5, C6, C7, C8, C9, J5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
