File: ethernet.kicad_sch (KiCad schematic)
At the start: 35 parts, among them J5 0826-1X1T-GJ-F, U2 LAN8742A, Y1 ECS-3225MVLC-500-CN-TR

Commit message: Started layout v2
Parts:
- D1: footprint WE-TVS_SOT23-6L_82402305:WE-TVS_SOT23-6L -> 82402305:WE-TVS_SOT23-6L
- J5: footprint 0826-1X1T-GJ-F:BEL_0826-1X1T-GJ-F -> 0826_1X1T_GJ_F:BEL_0826-1X1T-GJ-F
- L1: value L -> 2A/50mOhm
Connections:
- net at C10.2, D1.3, J5.11 (TRD1+)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: now also U2.20 (TXN); no longer U2.21 (TXP)
- net at C11.2, D1.1, J5.10 (TRD1-)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: now also U2.21 (TXP); no longer U2.20 (TXN)
- net at C13.2, J5.5 (TRD2-), R18.1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: now also D1.6; no longer D1.4
- net at C12.2, J5.4 (TRD2+), R19.1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: now also D1.4; no longer D1.6
Changed lines of the file:
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@@
 		)
 	)
+	(text_box "!IMPORTANT: LAN8742A supports polarity switching\nso we can switch TXP and TXN for easier routing\n(see datasheet p26)"
+		(exclude_from_sim no)
+		(at 168.91 57.15 0)
+		(size 24.13 16.51)
+		(margins 0.9525 0.9525 0.9525 0.9525)
+		(stroke
+			(width 0)
+			(type solid)
+		)
+		(fill
+			(type none)
+		)
+		(effects
+			(font
+				(size 1.27 1.27)
+			)
+			(justify left top)
+		)
+	)
 	(text_box "MODE[2:0]: internal PHY pull-ups present.\nExternal pull-ups added for robust reset strapping.\n\nMODE[2:0] = 111 ensures auto-negotiation mode"
 		(exclude_from_sim no)
@@
 	)
 	(junction
-		(at 196.85 62.23)
+		(at 191.77 83.82)
 		(diameter 0)
-		(color 194 194 0 1)
+		(color 0 0 0 0)
 	)
 	(junction
@@
 	)
 	(junction
+		(at 194.31 62.23)
+		(diameter 0)
+		(color 0 0 0 0)
+	)
+	(junction
 		(at 138.43 77.47)
 		(diameter 0)
@@
 	)
 	(junction
-		(at 191.77 81.28)
-		(diameter 0)
-		(color 0 0 0 0)
-	)
-	(junction
 		(at 109.22 27.94)
 		(diameter 0)
@@
 	)
 	(junction
+		(at 194.31 59.69)
+		(diameter 0)
+		(color 0 0 0 0)
+	)
+	(junction
 		(at 119.38 45.72)
 		(diameter 0)
@@
 	)
 	(junction
-		(at 194.31 62.23)
-		(diameter 0)
-		(color 194 194 0 1)
-	)
-	(junction
 		(at 129.54 96.52)
 		(diameter 0)
@@
 	)
 	(junction
-		(at 196.85 83.82)
-		(diameter 0)
-		(color 0 0 0 0)
-	)
-	(junction
 		(at 67.31 76.2)
 		(diameter 0)
@@
 	)
 	(junction
+		(at 196.85 81.28)
+		(diameter 0)
+		(color 0 0 0 0)
+	)
+	(junction
 		(at 147.32 81.28)
 		(diameter 0)
@@
 	(wire
 		(pts
-			(xy 168.91 105.41) (xy 168.91 95.25)
+			(xy 168.91 100.33) (xy 168.91 95.25)
 		)
 		(stroke
@@
 	(wire
 		(pts
-			(xy 196.85 59.69) (xy 196.85 62.23)
-		)
-		(stroke
-			(width 0.3048)
-			(type default)
-			(color 194 194 0 1)
-		)
-	)
-	(wire
-		(pts
 			(xy 148.59 62.23) (xy 157.48 62.23)
 		)
@@
 	(wire
 		(pts
-			(xy 194.31 62.23) (xy 196.85 62.23)
-		)
-		(stroke
-			(width 0.3048)
-			(type default)
-			(color 194 194 0 1)
-		)
-	)
-	(wire
-		(pts
 			(xy 44.45 128.27) (xy 46.99 128.27)
 		)
@@
 	(wire
 		(pts
+			(xy 157.48 54.61) (xy 157.48 62.23)
+		)
+		(stroke
+			(width 0.3048)
+			(type default)
+			(color 194 194 0 1)
+		)
+	)
+	(wire
+		(pts
 			(xy 106.68 148.59) (xy 127 148.59)
 		)
@@
 	(wire
 		(pts
+			(xy 191.77 83.82) (xy 191.77 92.71)
+		)
+		(stroke
+			(width 0)
+			(type default)
+		)
+	)
+	(wire
+		(pts
 			(xy 147.32 81.28) (xy 147.32 88.9)
 		)
@@
 	(wire
 		(pts
-			(xy 196.85 83.82) (xy 199.39 83.82)
+			(xy 191.77 83.82) (xy 199.39 83.82)
 		)
 		(stroke
@@
 	(wire
 		(pts
+			(xy 194.31 62.23) (xy 199.39 62.23)
+		)
+		(stroke
+			(width 0.3048)
+			(type default)
+			(color 194 194 0 1)
+		)
+	)
+	(wire
+		(pts
 			(xy 124.46 81.28) (xy 147.32 81.28)
 		)
@@
 	(wire
 		(pts
-			(xy 85.09 88.9) (xy 85.09 69.85)
+			(xy 194.31 54.61) (xy 194.31 59.69)
 		)
 		(stroke
-			(width 0)
+			(width 0.3048)
 			(type default)
+			(color 194 194 0 1)
 		)
 	)
 	(wire
 		(pts
-			(xy 142.24 111.76) (xy 156.21 111.76)
+			(xy 85.09 88.9) (xy 85.09 69.85)
 		)
 		(stroke
-			(width 0.3048)
+			(width 0)
 			(type default)
-			(color 255 0 0 1)
 		)
 	)
 	(wire
 		(pts
-			(xy 148.59 81.28) (xy 191.77 81.28)
+			(xy 142.24 111.76) (xy 156.21 111.76)
 		)
 		(stroke
-			(width 0)
+			(width 0.3048)
 			(type default)
+			(color 255 0 0 1)
 		)
 	)
@@
 	(wire
 		(pts
-			(xy 157.48 83.82) (xy 196.85 83.82)
+			(xy 157.48 83.82) (xy 191.77 83.82)
 		)
 		(stroke
@@
 	(wire
 		(pts
-			(xy 194.31 95.25) (xy 194.31 62.23)
-		)
-		(stroke
-			(width 0.3048)
-			(type default)
-			(color 194 194 0 1)
-		)
-	)
-	(wire
-		(pts
 			(xy 175.26 92.71) (xy 173.99 92.71)
 		)
@@
 	(wire
 		(pts
-			(xy 102.87 38.1) (xy 102.87 39.37)
+			(xy 194.31 59.69) (xy 199.39 59.69)
 		)
 		(stroke
 			(width 0.3048)
 			(type default)
-			(color 0 0 0 1)
+			(color 194 194 0 1)
 		)
 	)
 	(wire
 		(pts
-			(xy 135.89 133.35) (xy 142.24 133.35)
+			(xy 102.87 38.1) (xy 102.87 39.37)
 		)
 		(stroke
-			(width 0)
+			(width 0.3048)
 			(type default)
+			(color 0 0 0 1)
 		)
 	)
 	(wire
 		(pts
-			(xy 196.85 97.79) (xy 196.85 83.82)
+			(xy 135.89 133.35) (xy 142.24 133.35)
 		)
 		(stroke
@@
 	(wire
 		(pts
-			(xy 191.77 81.28) (xy 199.39 81.28)
+			(xy 148.59 81.28) (xy 196.85 81.28)
 		)
 		(stroke
@@
 	(wire
 		(pts
+			(xy 194.31 59.69) (xy 194.31 62.23)
+		)
+		(stroke
+			(width 0.3048)
+			(type default)
+			(color 194 194 0 1)
+		)
+	)
+	(wire
+		(pts
 			(xy 67.31 59.69) (xy 67.31 62.23)
 		)
@@
 	(wire
 		(pts
-			(xy 191.77 81.28) (xy 191.77 92.71)
-		)
-		(stroke
-			(width 0)
-			(type default)
-		)
-	)
-	(wire
-		(pts
 			(xy 44.45 135.89) (xy 44.45 138.43)
 		)
@@
 	(wire
 		(pts
-			(xy 157.48 62.23) (xy 194.31 62.23)
+			(xy 130.81 52.07) (xy 130.81 53.34)
 		)
 		(stroke
 			(width 0.3048)
 			(type default)
-			(color 194 194 0 1)
+			(color 0 0 0 1)
 		)
 	)
 	(wire
 		(pts
-			(xy 130.81 52.07) (xy 130.81 53.34)
+			(xy 233.68 125.73) (xy 236.22 125.73)
 		)
 		(stroke
-			(width 0.3048)
+			(width 0)
 			(type default)
-			(color 0 0 0 1)
 		)
 	)
 	(wire
 		(pts
-			(xy 233.68 125.73) (xy 236.22 125.73)
+			(xy 148.59 72.39) (xy 148.59 81.28)
 		)
 		(stroke
@@
 	(wire
 		(pts
-			(xy 148.59 72.39) (xy 148.59 81.28)
+			(xy 73.66 88.9) (xy 85.09 88.9)
 		)
 		(stroke
@@
 	(wire
 		(pts
-			(xy 196.85 62.23) (xy 199.39 62.23)
+			(xy 157.48 54.61) (xy 194.31 54.61)
 		)
 		(stroke
@@
 	(wire
 		(pts
-			(xy 73.66 88.9) (xy 85.09 88.9)
+			(xy 194.31 62.23) (xy 194.31 95.25)
 		)
 		(stroke
-			(width 0)
+			(width 0.3048)
 			(type default)
+			(color 194 194 0 1)
 		)
 	)
@@
 	(wire
 		(pts
+			(xy 196.85 81.28) (xy 196.85 97.79)
+		)
+		(stroke
+			(width 0)
+			(type default)
+		)
+	)
+	(wire
+		(pts
 			(xy 142.24 142.24) (xy 142.24 143.51)
 		)
@@
 	(wire
 		(pts
+			(xy 196.85 81.28) (xy 199.39 81.28)
+		)
+		(stroke
+			(width 0)
+			(type default)
+		)
+	)
+	(wire
+		(pts
 			(xy 102.87 30.48) (xy 92.71 30.48)
 		)
@@
 		)
 	)
-	(wire
-		(pts
-			(xy 199.39 59.69) (xy 196.85 59.69)
-		)
-		(stroke
-			(width 0.3048)
-			(type default)
-			(color 194 194 0 1)
-		)
-	)
 	(label "VDDA"
 		(at 132.08 27.94 0)
@@
 			)
 		)
-		(property "Value" "L"
+		(property "Value" "2A/50mOhm"
 			(at 124.46 25.4 90)
 			(effects
@@
 	(symbol
 		(lib_id "power:GND")
-		(at 168.91 105.41 0)
+		(at 168.91 100.33 0)
 		(unit 1)
 		(exclude_from_sim no)
@@
 		(dnp no)
 		(property "Reference" "#PWR02"
-			(at 168.91 111.76 0)
+			(at 168.91 106.68 0)
 			(effects
 				(font
@@
 		)
 		(property "Value" "GND"
-			(at 168.91 109.22 0)
+			(at 168.91 104.14 0)
 			(effects
 				(font
@@
 		)
 		(property "Footprint" ""
-			(at 168.91 105.41 0)
+			(at 168.91 100.33 0)
 			(effects
 				(font
@@
 		)
 		(property "Datasheet" ""
-			(at 168.91 105.41 0)
+			(at 168.91 100.33 0)
 			(effects
 				(font
@@
 		)
 		(property "Description" "Power symbol creates a global label with name \"GND\" , ground"
-			(at 168.91 105.41 0)
+			(at 168.91 100.33 0)
 			(effects
 				(font
@@
 			)
 		)
-		(property "Footprint" "WE-TVS_SOT23-6L_82402305:WE-TVS_SOT23-6L"
+		(property "Footprint" "82402305:WE-TVS_SOT23-6L"
 			(at 182.88 95.25 0)
 			(effects
@@
 			)
 		)
-		(property "Footprint" "0826-1X1T-GJ-F:BEL_0826-1X1T-GJ-F"
+		(property "Footprint" "0826_1X1T_GJ_F:BEL_0826-1X1T-GJ-F"
 			(at 220.98 85.09 0)
 			(effects
