File: miniServer.kicad_sch (KiCad schematic)
At the start: 31 parts, among them J10 Conn_01x01, J3 Conn_ARM_SWD_TagConnect_TC203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, U1 STM32H725VGTx, U5 NCP1117-3.3_SOT223

Commit message: Changed PowerSupply idea: use jumper to select PoE or VBUS
Parts:
- removed C16, C17: 10uF, Capacitor_SMD:C_0805_2012Metric_Pad1.18x1.45mm_HandSolder, symbol Device:C
- removed U5: NCP1117-3.3_SOT223, Package_TO_SOT_SMD:SOT-223-3_TabPin2, symbol Regulator_Linear:NCP1117-3.3_SOT223
Other:
- added sheet Power (power.kicad_sch)
- note removed: "Power"
- moved on the sheet: C18, C19, C20, C21, C22, C23, C25, C26, C27, C28, C33, C34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

Commit message: Started layout v2
Other:
- moved on the sheet: H1, H2, H3, H4
